Commit message: 加入四轮差速控制插件（两论差速控制插件），可通过键盘其控制

File: src/car_description/urdf/car.gazebo.xacro (robot description, xacro)
@@ -2,5 +2,5 @@
 <robot xmlns:xacro="http://www.ros.org/wiki/xacro">
 <xacro:macro name="car_gazebo">
-  <!-- 车身 -->
+  <!-- 车身物理与材质 -->
   <gazebo reference="base_link">
     <material>Gazebo/Blue</material>
@@ -10,5 +10,5 @@
     <mu2>1.0</mu2>
   </gazebo>
-  <!-- 四个轮子 -->
+  <!-- 左前轮 -->
   <gazebo reference="left_front_wheel_link">
     <material>Gazebo/Black</material>
@@ -19,4 +19,5 @@
     <minDepth>0.001</minDepth>
   </gazebo>
+  <!-- 右前轮 -->
   <gazebo reference="right_front_wheel_link">
     <material>Gazebo/Black</material>
@@ -26,4 +27,5 @@
     <mu2>10.0</mu2>
   </gazebo>
+  <!-- 左后轮 -->
   <gazebo reference="left_back_wheel_link">
     <material>Gazebo/Black</material>
@@ -33,4 +35,5 @@
     <mu2>10.0</mu2>
   </gazebo>
+  <!-- 右后轮 -->
   <gazebo reference="right_back_wheel_link">
     <material>Gazebo/Black</material>
@@ -44,5 +47,5 @@
     <material>Gazebo/Red</material>
   </gazebo>
-  <!-- 相机 -->
+  <!-- 深度相机 -->
   <gazebo reference="depth_camera_link">
     <material>Gazebo/Yellow</material>
@@ -52,4 +55,52 @@
     <material>Gazebo/Gray</material>
   </gazebo>
+  <!-- 四轮差速驱动插件 -->
+  <gazebo>
+    <plugin name="four_wheel_diff_drive" filename="libgazebo_ros_diff_drive.so">
+      <ros>
+        <namespace>/</namespace>
+        <remapping>cmd_vel:=/cmd_vel</remapping>
+        <remapping>odom:=/odom</remapping>
+      </ros>
+      <!-- 2对车轮 = 四轮驱动 -->
+      <num_wheel_pairs>2</num_wheel_pairs>
+      <!-- 第1对：前轮 -->
+      <left_joint>left_front_wheel_joint</left_joint>
+      <right_joint>right_front_wheel_joint</right_joint>
+      <!-- 第2对：后轮 -->
+      <left_joint>left_back_wheel_joint</left_joint>
+      <right_joint>right_back_wheel_joint</right_joint>
+      <!-- 轮距、轮径（和你模型匹配） -->
+      <wheel_separation>0.104</wheel_separation>
+      <wheel_diameter>0.12</wheel_diameter>
+      <wheel_separation_multiplier>1.0</wheel_separation_multiplier>
+      <wheel_radius_multiplier>1.0</wheel_radius_multiplier>
+      <!-- 运动限制 -->
+      <max_wheel_torque>20.0</max_wheel_torque>
+      <max_wheel_acceleration>5.0</max_wheel_acceleration>
+      <max_linear_speed>1.0</max_linear_speed>
+      <max_angular_speed>2.0</max_angular_speed>
+      <!-- 里程计 & TF 发布 -->
+      <publish_odom>true</publish_odom>
+      <publish_odom_tf>true</publish_odom_tf>
+      <odometry_frame>odom</odometry_frame>
+      <robot_base_frame>base_footprint</robot_base_frame>
+      <odometry_publish_rate>30.0</odometry_publish_rate>
+      <!-- 关键：开启关节状态发布 --><!-- 差速插件自身发布关节状态 -->
+      <publish_joint_states>true</publish_joint_states>
+      <joint_states_topic>joint_states</joint_states_topic>
+    </plugin>
+     <!-- 独立关节状态发布插件：兜底输出所有车轮关节数据 -->
+    <plugin name="car_joint_state" filename="libgazebo_ros_joint_state_publisher.so">
+      <ros>
+        <remapping>~/out:=joint_states</remapping>
+      </ros>
+      <update_rate>30</update_rate>
+      <joint_name>left_front_wheel_joint</joint_name>
+      <joint_name>right_front_wheel_joint</joint_name>
+      <joint_name>left_back_wheel_joint</joint_name>
+      <joint_name>right_back_wheel_joint</joint_name>
+    </plugin>
+  </gazebo>
 </xacro:macro>
 </robot>

File: src/car_description/urdf/car_base.urdf.xacro (robot description, xacro)
@@ -119,5 +119,5 @@
       <child link="left_front_wheel_link"/>
       <origin xyz="0.25  0.052  0" rpy="1.5708 0 0"/>
-      <axis xyz="0 0 1" />
+      <axis xyz="0 0 -1" />
   </joint>
   <!-- 右前轮 -->
@@ -126,5 +126,5 @@
       <child link="right_front_wheel_link"/>
       <origin xyz="0.25 -0.052  0" rpy="1.5708 0 0"/>
-      <axis xyz="0 0 1" />
+      <axis xyz="0 0 -1" />
   </joint>
   <!-- 左后轮 -->
@@ -133,5 +133,5 @@
       <child link="left_back_wheel_link"/>
       <origin xyz="-0.25  0.052  0" rpy="1.5708 0 0"/>
-      <axis xyz="0 0 1" />
+      <axis xyz="0 0 -1" />
   </joint>
   <!-- 右后轮 -->
@@ -140,5 +140,5 @@
       <child link="right_back_wheel_link"/>
       <origin xyz="-0.25 -0.052  0" rpy="1.5708 0 0"/>
-      <axis xyz="0 0 1" />
+      <axis xyz="0 0 -1" />
   </joint>
   <!-- imu joint -->

File: src/car_description/urdf/car_physics.xacro (robot description, xacro)
@@ -3,5 +3,5 @@
 <!-- ======================
      基础物理宏定义
-     包含：碰撞 + 惯性 + 摩擦
+     包含：碰撞 + 惯性
 ======================= -->
 <xacro:macro name="base_physics">

Commit message: 增加雷达插件和imu插件 但在小车原地转弯时如果转弯速度rad/s大于1.5会产生抖动的拖影点云  解决办法：转弯速度小于1.5

File: src/car_description/urdf/car.gazebo.xacro (robot description, xacro)
@@ -55,4 +55,5 @@
     <material>Gazebo/Gray</material>
   </gazebo>
+  <!-- ============================================================-->
   <!-- 四轮差速驱动插件 -->
   <gazebo>
@@ -103,4 +104,121 @@
     </plugin>
   </gazebo>
+  <!-- ============================================================-->
+  <!-- IMU 仿真传感器 -->
+  <gazebo reference="imu_link">
+    <sensor name="imu_sensor" type="imu">
+      <always_on>true</always_on>
+      <update_rate>100</update_rate>
+      <visualize>false</visualize>
+      <body>imu_link</body>
+      <plugin filename="libgazebo_ros_imu_sensor.so" name="imu_plugin">
+        <ros>
+          <namespace>/</namespace>
+          <!-- 改为标准ROS2 IMU话题 imu/data -->
+          <remapping>~/out:=imu/data</remapping>
+        </ros>
+        <!-- 地面小车：以自身安装姿态为初始参考 -->
+        <initial_orientation_as_reference>true</initial_orientation_as_reference>
+        <!--描述 IMU姿态数据噪声可信度，管定位滤波-->
+        <orientation_covariance>1e-6 0 0  0 1e-6 0  0 0 1e-6</orientation_covariance>
+      </plugin>
+      <imu>
+        <angular_velocity>
+          <x>
+            <noise type="gaussian">
+              <mean>0.0</mean>
+              <stddev>2e-4</stddev>
+              <bias_mean>0.0000075</bias_mean>
+              <bias_stddev>0.0000008</bias_stddev>
+            </noise>
+          </x>
+          <y>
+            <noise type="gaussian">
+              <mean>0.0</mean>
+              <stddev>2e-4</stddev>
+              <bias_mean>0.0000075</bias_mean>
+              <bias_stddev>0.0000008</bias_stddev>
+            </noise>
+          </y>
+          <z>
+            <noise type="gaussian">
+              <mean>0.0</mean>
+              <stddev>2e-4</stddev>
+              <bias_mean>0.0000075</bias_mean>
+              <bias_stddev>0.0000008</bias_stddev>
+            </noise>
+          </z>
+        </angular_velocity>
+        <linear_acceleration>
+          <x>
+            <noise type="gaussian">
+              <mean>0.0</mean>
+              <stddev>1.7e-2</stddev>
+              <bias_mean>0.1</bias_mean>
+              <bias_stddev>0.001</bias_stddev>
+            </noise>
+          </x>
+          <y>
+            <noise type="gaussian">
+              <mean>0.0</mean>
+              <stddev>1.7e-2</stddev>
+              <bias_mean>0.1</bias_mean>
+              <bias_stddev>0.001</bias_stddev>
+            </noise>
+          </y>
+          <z>
+            <noise type="gaussian">
+              <mean>0.0</mean>
+              <stddev>1.7e-2</stddev>
+              <bias_mean>0.1</bias_mean>
+              <bias_stddev>0.001</bias_stddev>
+            </noise>
+          </z>
+        </linear_acceleration>
+      </imu>
+    </sensor>
+  </gazebo>
+  <!-- ============================================================-->
+  <!-- 激光雷达 仿真插件 -->
+  <gazebo reference="laser_link">
+    <sensor name="laser_sensor" type="ray">
+      <always_on>true</always_on>
+      <visualize>true</visualize>
+      <!-- 刷新频率改为10Hz，满足导航/SLAM需求 -->
+      <update_rate>10</update_rate>
+      <ray>
+        <scan>
+          <horizontal>
+            <samples>360</samples>
+            <resolution>1.0</resolution>
+            <min_angle>0.0</min_angle>
+            <max_angle>6.28</max_angle>
+          </horizontal>
+        </scan>
+        <range>
+        <!-- 过滤近距离车身/晃动杂点 -->
+          <min>0.15</min>
+          <max>3.5</max>
+          <resolution>0.015</resolution>
+        </range>
+        <!-- 模拟雷达测距高斯噪声 -->
+        <noise>
+          <type>gaussian</type>
+          <mean>0.0</mean>
+          <stddev>0.01</stddev>
+        </noise>
+      </ray>
+      <!-- ROS 雷达转换插件 -->
+      <plugin name="laserscan" filename="libgazebo_ros_ray_sensor.so">
+        <ros>
+          <remapping>~/out:=scan</remapping>
+        </ros>
+        <output_type>sensor_msgs/LaserScan</output_type>
+        <frame_name>laser_link</frame_name>
+        <!-- 额外：启用Gazebo内置滤波，抑制运动畸变 -->
+        <scan_filter>true</scan_filter>
+      </plugin>
+    </sensor>
+  </gazebo>
 </xacro:macro>
 </robot>

File: src/car_description/urdf/car_base.urdf.xacro (robot description, xacro)
@@ -106,5 +106,5 @@
       <parent link="base_footprint" />
       <child link="base_link" />
-      <origin xyz="0 0 0.06" />  <!-- 前后   左右  上下  等于轮子半径，刚好着地 -->
+      <origin xyz="0 0 0.09" />  <!-- 前后   左右  上下   -->
   </joint>
   <!-- 雷达和车身 joint -->
@@ -118,5 +118,6 @@
       <parent link="base_link"/>
       <child link="left_front_wheel_link"/>
-      <origin xyz="0.25  0.052  0" rpy="1.5708 0 0"/>
+      <!-- 关键改动：z轴从0改为-0.03，让轮胎整体下移3cm -->
+      <origin xyz="0.25  0.052  -0.03" rpy="1.5708 0 0"/>
       <axis xyz="0 0 -1" />
   </joint>
@@ -125,5 +126,6 @@
       <parent link="base_link"/>
       <child link="right_front_wheel_link"/>
-      <origin xyz="0.25 -0.052  0" rpy="1.5708 0 0"/>
+      <!-- 关键改动：z轴从0改为-0.03，让轮胎整体下移3cm -->
+      <origin xyz="0.25 -0.052  -0.03" rpy="1.5708 0 0"/>
       <axis xyz="0 0 -1" />
   </joint>
@@ -132,5 +134,6 @@
       <parent link="base_link"/>
       <child link="left_back_wheel_link"/>
-      <origin xyz="-0.25  0.052  0" rpy="1.5708 0 0"/>
+      <!-- 关键改动：z轴从0改为-0.03，让轮胎整体下移3cm -->
+      <origin xyz="-0.25  0.052  -0.03" rpy="1.5708 0 0"/>
       <axis xyz="0 0 -1" />
   </joint>
@@ -139,5 +142,6 @@
       <parent link="base_link"/>
       <child link="right_back_wheel_link"/>
-      <origin xyz="-0.25 -0.052  0" rpy="1.5708 0 0"/>
+      <!-- 关键改动：z轴从0改为-0.03，让轮胎整体下移3cm -->
+      <origin xyz="-0.25 -0.052  -0.03" rpy="1.5708 0 0"/>
       <axis xyz="0 0 -1" />
   </joint>

File: src/car_description/urdf/car_physics.xacro (robot description, xacro)
@@ -13,5 +13,5 @@
   </collision>
   <inertial>
-    <mass value="1.2"/>
+    <mass value="2.0"/> <!-- 1.2 -->
     <inertia ixx="0.01" ixy="0.0" ixz="0.0"
              iyy="0.08" iyz="0.0"

Commit message: 添加深度相机插件

File: src/car_description/urdf/car.gazebo.xacro (robot description, xacro)
@@ -221,4 +221,44 @@
     </sensor>
   </gazebo>
+  <!-- ============================================================-->
+  <!-- 深度相机 + RGB 相机 Gazebo 插件 -->
+  <gazebo reference="depth_camera_link">
+  <sensor type="depth" name="depth_camera">
+    <always_on>true</always_on>
+    <update_rate>15</update_rate>
+    <visualize>false</visualize>
+    <camera>
+      <horizontal_fov>1.047</horizontal_fov>
+      <image>
+        <width>640</width>
+        <height>480</height>
+        <format>R8G8B8</format>
+      </image>
+      <depth_camera>
+        <output>depth_image</output>
+      </depth_camera>
+      <clip>
+        <near>0.1</near>
+        <far>5.0</far>
+      </clip>
+      <noise>
+        <type>gaussian</type>
+        <mean>0.0</mean>
+        <stddev>0.01</stddev>
+      </noise>
+    </camera>
+    <!-- ROS2 通用相机插件（同时支持RGB+深度） -->
+        <plugin name="gazebo_ros_camera" filename="libgazebo_ros_camera.so">
+      <ros>
+        <!-- 关键：设置命名空间，统一话题前缀 -->
+        <remapping>~/image_raw:=image_raw</remapping>
+        <remapping>~/depth_image:=depth/image_raw</remapping>
+        <remapping>~/camera_info:=camera_info</remapping>
+      </ros>
+      <frame_name>camera_color_optical_frame</frame_name>
+      <depth>true</depth>
+    </plugin>
+  </sensor>
+</gazebo>
 </xacro:macro>
 </robot>

File: src/car_description/urdf/car_base.urdf.xacro (robot description, xacro)
@@ -93,5 +93,5 @@
       <!-- 相机外形：小长方体，尺寸可自行修改 -->
       <geometry>
-        <box size="0.09 0.02 0.02"/>
+        <box size="0.02 0.09 0.02"/>
       </geometry>
       <material name="yellow"/>
@@ -157,5 +157,12 @@
   <child link="depth_camera_link"/>
   <!-- x=0.375 车身总长0.75/2+相机厚度0.02/2；y=0居中；z=0.02 安装在车身前部下方 -->
-  <origin xyz="0.385 0 0.02" rpy="0 0 1.57"/>
+  <origin xyz="0.42 0 0.02" rpy="0 0 0"/>
+</joint>
+ <!-- 深度相机 虚拟坐标-->
+<link name="camera_color_optical_frame" />
+<joint name="camera_optical_joint" type="fixed">
+  <parent link="depth_camera_link"/>
+  <child link="camera_color_optical_frame"/>
+  <origin xyz="0 0 0" rpy="-1.5708 0 -1.5708"/>
 </joint>
 </robot>

File: src/car_description/urdf/car_physics.xacro (robot description, xacro)
@@ -69,12 +69,13 @@
     <origin xyz="0 0 0" rpy="0 0 0"/>
     <geometry>
-      <box size="0.09 0.02 0.02"/>
+      <box size="0.02 0.09 0.02"/>
     </geometry>
   </collision>
   <inertial>
     <mass value="0.08"/>
-    <inertia ixx="0.0001" ixy="0" ixz="0"
-             iyy="0.0005" iyz="0"
-             izz="0.0005"/>
+     <inertia
+      ixx="0.000034" ixy="0" ixz="0"
+      iyy="0.000017" iyz="0"
+      izz="0.000034"/>
   </inertial>
 </xacro:macro>

Commit message: 基本实现  地图建图 nav2导航  但是本电脑 仿真效率低 无法完整 跑完全部

File: src/car_description/urdf/car.gazebo.xacro (robot description, xacro)
@@ -76,10 +76,10 @@
       <wheel_diameter>0.12</wheel_diameter>
       <wheel_separation_multiplier>1.0</wheel_separation_multiplier>
-      <wheel_radius_multiplier>1.0</wheel_radius_multiplier>
+      <wheel_radius_multiplier>-1.0</wheel_radius_multiplier>
       <!-- 运动限制 -->
       <max_wheel_torque>20.0</max_wheel_torque>
-      <max_wheel_acceleration>5.0</max_wheel_acceleration>
-      <max_linear_speed>1.0</max_linear_speed>
-      <max_angular_speed>2.0</max_angular_speed>
+      <max_wheel_acceleration>50.0</max_wheel_acceleration><!-- 原来5.0→加速限制 -->
+      <max_linear_speed>1.8</max_linear_speed> <!-- 原本1.0 直行最大m/s-->
+      <max_angular_speed>3.0</max_angular_speed> <!-- 原来2.0→转弯最大rad/s -->
       <!-- 里程计 & TF 发布 -->
       <publish_odom>true</publish_odom>
@@ -184,5 +184,5 @@
     <sensor name="laser_sensor" type="ray">
       <always_on>true</always_on>
-      <visualize>true</visualize>
+      <visualize>false</visualize>
       <!-- 刷新频率改为10Hz，满足导航/SLAM需求 -->
       <update_rate>10</update_rate>

File: src/car_description/urdf/car_base.urdf.xacro (robot description, xacro)
@@ -119,6 +119,6 @@
       <child link="left_front_wheel_link"/>
       <!-- 关键改动：z轴从0改为-0.03，让轮胎整体下移3cm -->
-      <origin xyz="0.25  0.052  -0.03" rpy="1.5708 0 0"/>
-      <axis xyz="0 0 -1" />
+      <origin xyz="0.25  0.052  -0.03" rpy="-1.5708 0 0"/>
+      <axis xyz="0 0 1" />
   </joint>
   <!-- 右前轮 -->
@@ -127,6 +127,6 @@
       <child link="right_front_wheel_link"/>
       <!-- 关键改动：z轴从0改为-0.03，让轮胎整体下移3cm -->
-      <origin xyz="0.25 -0.052  -0.03" rpy="1.5708 0 0"/>
-      <axis xyz="0 0 -1" />
+      <origin xyz="0.25 -0.052  -0.03" rpy="-1.5708 0 0"/>
+      <axis xyz="0 0 1" />
   </joint>
   <!-- 左后轮 -->
@@ -135,6 +135,6 @@
       <child link="left_back_wheel_link"/>
       <!-- 关键改动：z轴从0改为-0.03，让轮胎整体下移3cm -->
-      <origin xyz="-0.25  0.052  -0.03" rpy="1.5708 0 0"/>
-      <axis xyz="0 0 -1" />
+      <origin xyz="-0.25  0.052  -0.03" rpy="-1.5708 0 0"/>
+      <axis xyz="0 0 1" />
   </joint>
   <!-- 右后轮 -->
@@ -143,6 +143,6 @@
       <child link="right_back_wheel_link"/>
       <!-- 关键改动：z轴从0改为-0.03，让轮胎整体下移3cm -->
-      <origin xyz="-0.25 -0.052  -0.03" rpy="1.5708 0 0"/>
-      <axis xyz="0 0 -1" />
+      <origin xyz="-0.25 -0.052  -0.03" rpy="-1.5708 0 0"/>
+      <axis xyz="0 0 1" />
   </joint>
   <!-- imu joint -->
@@ -150,5 +150,5 @@
       <parent link="base_link" />
       <child link="imu_link" />
-      <origin xyz="0 0 0.02" />
+      <origin xyz="0 0 0" />
   </joint>
   <!-- 深度相机 固定关节，安装在车头最前端 -->
